File: SHT4x_sub.kicad_sch (KiCad schematic)
At the start: 6 parts, among them J4 Conn_01x04_Pin, J5 Conn_01x04_Pin, U3 SHT4x

Commit message: sent to JLC noodleUSBp16
Other:
- moved on the sheet: C9, J4, J5
