File: SCPI_tempIO.kicad_sch (KiCad schematic)
At the start: 24 parts, among them J1 Conn_ARM_JTAG_SWD_10, J2 Conn_02x05_Counter_Clockwise, J3 USB_C_Receptacle_USB2.0_16P, SW1 SW_SPST, U1 STM32G0B1KBT6, U2 AP2112K-3.3

Commit message: schematic hotfix for VTref to VDD and note about Vref to VCC jumper on treedix board.
Connections:
- net 3v3: now also C7.1, J1.1 (VTref)
- net at J3.A4 (VBUS), J3.A9 (VBUS), J3.B4 (VBUS)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: no longer C7.1, J1.1 (VTref)
Other:
- note added: "HOTFIX! originally connected to VBUS, but should be mcu Vcc"
- note added: "note for Treedix.com JTAG/SWD adapter board, install VCC->VREF jumper. Otherwise ST-link will read Vref 1.7V, which means the pin is floating."
Changed lines of the file:
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@@
 		(company "nacho.works")
 	)
+	(text "HOTFIX! originally connected to VBUS,\n but should be mcu Vcc"
+		(exclude_from_sim no)
+		(at 74.93 71.882 90)
+		(effects
+			(font
+				(size 1.27 1.27)
+			)
+		)
+	)
+	(text "note for Treedix.com JTAG/SWD adapter board, \ninstall VCC->VREF jumper.\nOtherwise ST-link will read Vref 1.7V, \nwhich means the pin is floating.\n"
+		(exclude_from_sim no)
+		(at 26.416 130.048 0)
+		(effects
+			(font
+				(size 0.762 0.762)
+			)
+			(justify left)
+		)
+	)
 	(text "\nC5,C6,C9\nC49678\n100n\n0805\n\nC7\nC28323\n1u\n0805\n\nC8\nC1744\n4.7n\n0805\n\nD1\nC965793\nLED\n0402\n\nJ1\nC2935458\nConn_ARM_JTAG_SWD_10\nPinHeader_2x05_P1.27mm_Vertical_SMD\n\nJ3\nC963213\nUSB_C_Receptacle_USB2.0_16P\nUSB_C_Receptacle_G-Switch_GT-USB-7025\n\nR9\nC11702\n1000\n0402\n\nR10,R11\nC25905\n5.1k\n0402\n\nR12,R13\nC25092\n22\n0402\n\nR14,R15,R16,R17,R18,R19,R20,R21\nC25104\n330\n0402\n\nR23,R24\nC25744\n10k\n0402\n\nSW1\nC10852\nSW_SPST\nSW_Push_1P1T_NO_CK_KSC7xxJ\n\nU1\nC5270165\nST STM32G0B1KBT6\nLQFP-32_7x7mm_P0.8mm\n\nU2\nC23380830\nAP2112K-3.3\nSOT-23-5\n\nU3\nC54946589\nSHT4x\nSensirion_DFN-4_1.5x1.5mm_P0.8mm_SHT4x_NoCentralPad\n"
 		(exclude_from_sim no)
@@
 	)
 	(junction
-		(at 66.04 96.52)
+		(at 96.52 31.75)
 		(diameter 0)
 		(color 0 0 0 0)
 	)
 	(junction
-		(at 96.52 31.75)
+		(at 107.95 31.75)
 		(diameter 0)
 		(color 0 0 0 0)
 	)
 	(junction
-		(at 66.04 69.85)
+		(at 100.33 130.81)
 		(diameter 0)
 		(color 0 0 0 0)
 	)
 	(junction
-		(at 107.95 31.75)
+		(at 91.44 31.75)
 		(diameter 0)
 		(color 0 0 0 0)
 	)
 	(junction
-		(at 100.33 130.81)
+		(at 66.04 96.52)
 		(diameter 0)
 		(color 0 0 0 0)
@@
 	(wire
 		(pts
-			(xy 66.04 96.52) (xy 66.04 69.85)
+			(xy 72.39 34.29) (xy 69.85 34.29)
 		)
 		(stroke
@@
 	(wire
 		(pts
-			(xy 72.39 34.29) (xy 69.85 34.29)
+			(xy 97.79 130.81) (xy 100.33 130.81)
 		)
 		(stroke
@@
 	(wire
 		(pts
-			(xy 97.79 130.81) (xy 100.33 130.81)
+			(xy 154.94 77.47) (xy 166.37 77.47)
 		)
 		(stroke
@@
 	(wire
 		(pts
-			(xy 154.94 77.47) (xy 166.37 77.47)
+			(xy 74.93 93.98) (xy 74.93 49.53)
 		)
 		(stroke
 			(width 0)
-			(type default)
+			(type dash_dot)
+			(color 0 194 0 1)
 		)
 	)
@@
 	(wire
 		(pts
+			(xy 74.93 49.53) (xy 91.44 49.53)
+		)
+		(stroke
+			(width 0)
+			(type default)
+		)
+	)
+	(wire
+		(pts
 			(xy 266.7 54.61) (xy 266.7 90.17)
 		)
@@
 	(wire
 		(pts
+			(xy 66.04 93.98) (xy 74.93 93.98)
+		)
+		(stroke
+			(width 0)
+			(type default)
+		)
+	)
+	(wire
+		(pts
 			(xy 81.28 54.61) (xy 81.28 118.11)
 		)
@@
 	(wire
 		(pts
+			(xy 91.44 49.53) (xy 91.44 31.75)
+		)
+		(stroke
+			(width 0)
+			(type default)
+		)
+	)
+	(wire
+		(pts
 			(xy 193.04 90.17) (xy 193.04 72.39)
 		)
@@
 	(wire
 		(pts
+			(xy 66.04 96.52) (xy 66.04 93.98)
+		)
+		(stroke
+			(width 0)
+			(type default)
+		)
+	)
+	(wire
+		(pts
 			(xy 59.69 77.47) (xy 57.15 77.47)
 		)
@@
 	(wire
 		(pts
-			(xy 87.63 31.75) (xy 96.52 31.75)
+			(xy 87.63 31.75) (xy 91.44 31.75)
 		)
 		(stroke
@@
 	(wire
 		(pts
+			(xy 91.44 31.75) (xy 96.52 31.75)
+		)
+		(stroke
+			(width 0)
+			(type default)
+		)
+	)
+	(wire
+		(pts
 			(xy 62.23 82.55) (xy 55.88 82.55)
 		)
@@
 		)
 		(instances
-			(project "SCPI_tempIO-rounded"
+			(project "SCPI_tempIO"
 				(path "/3fa88ee0-2858-4485-b643-2061ac43b60a"
 					(reference "#PWR03")
@@
 		)
 		(instances
-			(project "SCPI_tempIO-rounded"
+			(project "SCPI_tempIO"
 				(path "/3fa88ee0-2858-4485-b643-2061ac43b60a"
 					(reference "#PWR02")
@@
 		)
 		(instances
-			(project "SCPI_tempIO-rounded"
+			(project "SCPI_tempIO"
 				(path "/3fa88ee0-2858-4485-b643-2061ac43b60a"
 					(reference "#PWR05")
@@
 		)
 		(instances
-			(project "SCPI_tempIO-rounded"
+			(project "SCPI_tempIO"
 				(path "/3fa88ee0-2858-4485-b643-2061ac43b60a"
 					(reference "#PWR04")
@@
 		)
 		(instances
-			(project "SCPI_tempIO-rounded"
+			(project "SCPI_tempIO"
 				(path "/3fa88ee0-2858-4485-b643-2061ac43b60a"
 					(reference "#PWR01")
@@
 		)
 		(instances
-			(project "SCPI_tempIO-rounded"
+			(project "SCPI_tempIO"
 				(path "/3fa88ee0-2858-4485-b643-2061ac43b60a"
 					(reference "SW1")
@@
 		)
 		(instances
-			(project "SCPI_tempIO-rounded"
+			(project "SCPI_tempIO"
 				(path "/3fa88ee0-2858-4485-b643-2061ac43b60a"
 					(reference "R10")
@@
 		)
 		(instances
-			(project "SCPI_tempIO-rounded"
+			(project "SCPI_tempIO"
 				(path "/3fa88ee0-2858-4485-b643-2061ac43b60a"
 					(reference "U1")
@@
 		)
 		(instances
-			(project "SCPI_tempIO-rounded"
+			(project "SCPI_tempIO"
 				(path "/3fa88ee0-2858-4485-b643-2061ac43b60a"
 					(reference "R15")
@@
 		)
 		(instances
-			(project "SCPI_tempIO-rounded"
+			(project "SCPI_tempIO"
 				(path "/3fa88ee0-2858-4485-b643-2061ac43b60a"
 					(reference "C8")
@@
 		)
 		(instances
-			(project "SCPI_tempIO-rounded"
+			(project "SCPI_tempIO"
 				(path "/3fa88ee0-2858-4485-b643-2061ac43b60a"
 					(reference "C5")
@@
 		)
 		(instances
-			(project "SCPI_tempIO-rounded"
+			(project "SCPI_tempIO"
 				(path "/3fa88ee0-2858-4485-b643-2061ac43b60a"
 					(reference "#PWR011")
@@
 		)
 		(instances
-			(project "SCPI_tempIO-rounded"
+			(project "SCPI_tempIO"
 				(path "/3fa88ee0-2858-4485-b643-2061ac43b60a"
 					(reference "C7")
@@
 		)
 		(instances
-			(project "SCPI_tempIO-rounded"
+			(project "SCPI_tempIO"
 				(path "/3fa88ee0-2858-4485-b643-2061ac43b60a"
 					(reference "R12")
@@
 		)
 		(instances
-			(project "SCPI_tempIO-rounded"
+			(project "SCPI_tempIO"
 				(path "/3fa88ee0-2858-4485-b643-2061ac43b60a"
 					(reference "R17")
@@
 		)
 		(instances
-			(project "SCPI_tempIO-rounded"
+			(project "SCPI_tempIO"
 				(path "/3fa88ee0-2858-4485-b643-2061ac43b60a"
 					(reference "C6")
@@
 		)
 		(instances
-			(project "SCPI_tempIO-rounded"
+			(project "SCPI_tempIO"
 				(path "/3fa88ee0-2858-4485-b643-2061ac43b60a"
 					(reference "R11")
@@
 		)
 		(instances
-			(project "SCPI_tempIO-rounded"
+			(project "SCPI_tempIO"
 				(path "/3fa88ee0-2858-4485-b643-2061ac43b60a"
 					(reference "R18")
@@
 		)
 		(instances
-			(project "SCPI_tempIO-rounded"
+			(project "SCPI_tempIO"
 				(path "/3fa88ee0-2858-4485-b643-2061ac43b60a"
 					(reference "R16")
@@
 		)
 		(instances
-			(project "SCPI_tempIO-rounded"
+			(project "SCPI_tempIO"
 				(path "/3fa88ee0-2858-4485-b643-2061ac43b60a"
 					(reference "#PWR014")
@@
 		)
 		(instances
-			(project "SCPI_tempIO-rounded"
+			(project "SCPI_tempIO"
 				(path "/3fa88ee0-2858-4485-b643-2061ac43b60a"
 					(reference "#PWR010")
@@
 		)
 		(instances
-			(project "SCPI_tempIO-rounded"
+			(project "SCPI_tempIO"
 				(path "/3fa88ee0-2858-4485-b643-2061ac43b60a"
 					(reference "#PWR09")
@@
 		)
 		(instances
-			(project "SCPI_tempIO-rounded"
+			(project "SCPI_tempIO"
 				(path "/3fa88ee0-2858-4485-b643-2061ac43b60a"
 					(reference "R20")
@@
 		)
 		(instances
-			(project "SCPI_tempIO-rounded"
+			(project "SCPI_tempIO"
 				(path "/3fa88ee0-2858-4485-b643-2061ac43b60a"
 					(reference "J1")
@@
 		)
 		(instances
-			(project "SCPI_tempIO-rounded"
+			(project "SCPI_tempIO"
 				(path "/3fa88ee0-2858-4485-b643-2061ac43b60a"
 					(reference "R13")
@@
 		)
 		(instances
-			(project "SCPI_tempIO-rounded"
+			(project "SCPI_tempIO"
 				(path "/3fa88ee0-2858-4485-b643-2061ac43b60a"
 					(reference "R9")
@@
 		)
 		(instances
-			(project "SCPI_tempIO-rounded"
+			(project "SCPI_tempIO"
 				(path "/3fa88ee0-2858-4485-b643-2061ac43b60a"
 					(reference "R14")
@@
 		)
 		(instances
-			(project "SCPI_tempIO-rounded"
+			(project "SCPI_tempIO"
 				(path "/3fa88ee0-2858-4485-b643-2061ac43b60a"
 					(reference "D1")
@@
 		)
 		(instances
-			(project "SCPI_tempIO-rounded"
+			(project "SCPI_tempIO"
 				(path "/3fa88ee0-2858-4485-b643-2061ac43b60a"
 					(reference "#PWR015")
@@
 		)
 		(instances
-			(project "SCPI_tempIO-rounded"
+			(project "SCPI_tempIO"
 				(path "/3fa88ee0-2858-4485-b643-2061ac43b60a"
 					(reference "R21")
@@
 		(in_pos_files yes)
 		(dnp no)
-		(fields_autoplaced yes)
 		(property "Reference" "#PWR08"
 			(at 100.33 138.43 0)
@@
 		)
 		(property "Value" "GND"
-			(at 100.33 137.16 0)
+			(at 103.124 132.08 0)
 			(show_name no)
 			(do_not_autoplace no)
@@
 		)
 		(instances
-			(project "SCPI_tempIO-rounded"
+			(project "SCPI_tempIO"
 				(path "/3fa88ee0-2858-4485-b643-2061ac43b60a"
 					(reference "#PWR08")
@@
 		)
 		(instances
-			(project "SCPI_tempIO-rounded"
+			(project "SCPI_tempIO"
 				(path "/3fa88ee0-2858-4485-b643-2061ac43b60a"
 					(reference "U2")
@@
 		)
 		(instances
-			(project "SCPI_tempIO-rounded"
+			(project "SCPI_tempIO"
 				(path "/3fa88ee0-2858-4485-b643-2061ac43b60a"
 					(reference "J3")
@@
 		)
 		(instances
-			(project "SCPI_tempIO-rounded"
+			(project "SCPI_tempIO"
 				(path "/3fa88ee0-2858-4485-b643-2061ac43b60a"
 					(reference "#PWR07")
@@
 		)
 		(instances
-			(project "SCPI_tempIO-rounded"
+			(project "SCPI_tempIO"
 				(path "/3fa88ee0-2858-4485-b643-2061ac43b60a"
 					(reference "J2")
@@
 		)
 		(instances
-			(project "SCPI_tempIO-rounded"
+			(project "SCPI_tempIO"
 				(path "/3fa88ee0-2858-4485-b643-2061ac43b60a"
 					(reference "#PWR013")
@@
 		)
 		(instances
-			(project "SCPI_tempIO-rounded"
+			(project "SCPI_tempIO"
 				(path "/3fa88ee0-2858-4485-b643-2061ac43b60a"
 					(reference "R19")
@@
 		)
 		(instances
-			(project "SCPI_tempIO-rounded"
+			(project "SCPI_tempIO"
 				(path "/3fa88ee0-2858-4485-b643-2061ac43b60a"
 					(page "2")
