File: hardware/SCPI_tempIO.kicad_pcb (KiCad board)
At the start: 2 copper layers, 42.6 x 22.2 mm, 31 parts, among them J1 Conn_ARM_JTAG_SWD_10, J2 Conn_02x05_Counter_Clockwise, J3 USB_C_Receptacle_USB2.0_14P, J4 Conn_01x04_Pin, J5 Conn_01x04_Pin, SW1 SW_SPST, U1 STM32G070KBTx, U2 AP2112K-3.3, U3 SHT4x

Commit message: Hardware: make the rounded (fabricated) board the project PCB
SCPI_tempIO-rounded.kicad_pcb replaces SCPI_tempIO.kicad_pcb, which was the
pre-rounding board with the old HRO USB-C connector. One project now, so
Update PCB from Schematic works. The rounded project's extra 0.1 mm track
width is carried over; its .kicad_pro/.kicad_dru are removed.

Co-Authored-By: Claude Opus 5.5 <noreply@anthropic.com>
Parts:
- J3: value USB_C_Receptacle_USB2.0_14P -> USB_C_Receptacle_USB2.0_16P; footprint Connector_USB:USB_C_Receptacle_HRO_TYPE-C-31-M-12 -> Connector_USB:USB_C_Receptacle_G-Switch_GT-USB-7025
- moved J3 0.59 mm to (64.8, 44.8)
Connections:
- J3 pad A8: (no net) -> unconnected-(J3-SBU1-PadA8)
- J3 pad B8: (no net) -> unconnected-(J3-SBU2-PadB8)
Routing:
- net /3v3: track 58.4 -> 50.7 mm
- net Net-(J3-D--PadA7): track 11.5 -> 14.4 mm, vias 0 -> 2
- net GND: track 28.7 -> 30.2 mm, vias 24 -> 25
- net Net-(J1-~{RESET}): track 23.7 -> 22.4 mm
- net Net-(J1-VTref): track 27.0 -> 25.7 mm
- net Net-(J3-CC2): track 1.71 -> 2.76 mm
- net Net-(J3-CC1): track 1.85 -> 2.66 mm
- added copper zone on F.Cu, net /3v3
